File: board/kicad/nantor.kicad_pcb (KiCad board)
At the start: 2 copper layers, 139.5 x 94.4 mm, 26 parts, among them J1 Bridge, J2 Batt, SW1 Power, SW2 Power, U1 YAAJ_WeAct_BlackPill_Part_Like

Commit message: Make switch open
Connections:
- SW1 pad 3: GND -> unconnected-(SW1-C-Pad3)
- SW2 pad 1: GND -> unconnected-(SW2-A-Pad1)
Changed lines of the file:
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@@
   (net 38 "unconnected-(U1-PB2-Pad36)")
   (net 39 "unconnected-(U1-5V-Pad40)")
+  (net 40 "unconnected-(SW1-C-Pad3)")
+  (net 41 "unconnected-(SW2-A-Pad1)")
   (footprint "nantor:Kailh_socket_PG1350_optional_reversible_clean" (layer "F.Cu")
     (at 168.506983 81.277968)
@@
       (net 24 "Net-(SW1-B)") (pinfunction "B") (pintype "passive"))
     (pad "3" smd rect (at 2.25 -1.43 90) (size 0.7 1.5) (layers "F.Cu" "F.Paste" "F.Mask")
-      (net 2 "GND") (pinfunction "C") (pintype "passive"))
+      (net 40 "unconnected-(SW1-C-Pad3)") (pinfunction "C") (pintype "passive+no_connect"))
     (model "${KICAD6_3DMODEL_DIR}/Button_Switch_SMD.3dshapes/SW_SPDT_PCM12.wrl"
       (offset (xyz 0 0 0))
@@
     (pad "" smd rect (at 3.65 0.78 270) (size 1 0.8) (layers "B.Cu" "B.Paste" "B.Mask"))
     (pad "1" smd rect (at -2.25 1.43 270) (size 0.7 1.5) (layers "B.Cu" "B.Paste" "B.Mask")
-      (net 2 "GND") (pinfunction "A") (pintype "passive"))
+      (net 41 "unconnected-(SW2-A-Pad1)") (pinfunction "A") (pintype "passive+no_connect"))
     (pad "2" smd rect (at 0.75 1.43 270) (size 0.7 1.5) (layers "B.Cu" "B.Paste" "B.Mask")
       (net 24 "Net-(SW1-B)") (pinfunction "B") (pintype "passive"))
