File: board/kicad/nantor.kicad_sch (KiCad schematic)
At the start: 26 parts, among them J1 Bridge, J2 Batt, SW1 Power, SW2 Power, U1 YAAJ_WeAct_BlackPill_Part_Like

Commit message: Make switch open
Connections:
- net GND: no longer SW1.3 (C), SW2.1 (A)
- net at U1.14 (PB6): now also J1.TX; no longer J1.R2
- net at U1.15 (PB7): now also J1.RX; no longer J1.R1
- no-connect marks 12 -> 14
Changed lines of the file:
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@@
 (kicad_sch (version 20230121) (generator eeschema)
   (paper "A4")
-  (junction (at 205.74 113.03) (diameter 0) (color 0 0 0 0)
-  )
   (junction (at 187.96 105.41) (diameter 0) (color 0 0 0 0)
   )
@@
   (no_connect (at 232.41 50.8))
   (no_connect (at 232.41 58.42))
+  (no_connect (at 207.01 107.95))
   (no_connect (at 232.41 81.28))
   (no_connect (at 189.23 38.1))
@@
   (no_connect (at 232.41 53.34))
   (no_connect (at 189.23 83.82))
+  (no_connect (at 207.01 119.38))
   (no_connect (at 189.23 48.26))
   (no_connect (at 189.23 76.2))
@@
     (stroke (width 0) (type default))
   )
-  (wire (pts (xy 205.74 113.03) (xy 209.55 113.03))
-    (stroke (width 0) (type default))
-  )
   (wire (pts (xy 184.15 66.04) (xy 190.5 66.04))
     (stroke (width 0) (type default))
@@
     (stroke (width 0) (type default))
   )
+  (wire (pts (xy 204.47 119.38) (xy 207.01 119.38))
+    (stroke (width 0) (type default))
+  )
   (wire (pts (xy 125.73 92.71) (xy 125.73 90.17))
     (stroke (width 0) (type default))
@@
     (stroke (width 0) (type default))
   )
-  (wire (pts (xy 205.74 119.38) (xy 205.74 113.03))
-    (stroke (width 0) (type default))
-  )
   (wire (pts (xy 125.73 107.95) (xy 123.19 107.95))
     (stroke (width 0) (type default))
@@
     (stroke (width 0) (type default))
   )
-  (wire (pts (xy 204.47 119.38) (xy 205.74 119.38))
-    (stroke (width 0) (type default))
-  )
   (wire (pts (xy 248.92 76.2) (xy 246.38 76.2))
     (stroke (width 0) (type default))
@@
     (stroke (width 0) (type default))
   )
-  (wire (pts (xy 205.74 107.95) (xy 205.74 113.03))
-    (stroke (width 0) (type default))
-  )
   (wire (pts (xy 231.14 55.88) (xy 232.41 55.88))
     (stroke (width 0) (type default))
@@
     (stroke (width 0) (type default))
   )
-  (wire (pts (xy 205.74 107.95) (xy 204.47 107.95))
+  (wire (pts (xy 204.47 107.95) (xy 207.01 107.95))
     (stroke (width 0) (type default))
   )
@@
   )
   (wire (pts (xy 82.55 90.17) (xy 80.01 90.17))
-    (stroke (width 0) (type default))
-  )
-  (wire (pts (xy 209.55 113.03) (xy 209.55 118.11))
     (stroke (width 0) (type default))
   )
@@
     )
   )
-  (symbol (lib_id "power:GND") (at 209.55 118.11 0) (unit 1)
-    (in_bom yes) (on_board yes) (dnp no) (fields_autoplaced)
-    (property "Reference" "#PWR01" (at 209.55 124.46 0)
-      (effects (font (size 1.27 1.27)) hide)
-    )
-    (property "Value" "GND" (at 209.55 123.19 0)
-      (effects (font (size 1.27 1.27)))
-    )
-    (property "Footprint" "" (at 209.55 118.11 0)
-      (effects (font (size 1.27 1.27)) hide)
-    )
-    (property "Datasheet" "" (at 209.55 118.11 0)
-      (effects (font (size 1.27 1.27)) hide)
-    )
-    (pin "1")
-    (instances
-      (project "nantor"
-        (path "/3ca8fd45-5a9e-4ec9-b4a3-11c42137b74e"
-          (reference "#PWR01") (unit 1)
-        )
-      )
-    )
-  )
   (symbol (lib_id "Switch:SW_Push") (at 96.52 125.73 0) (unit 1)
     (in_bom yes) (on_board yes) (dnp no) (fields_autoplaced)
@@
   (symbol (lib_id "Connector_Audio:AudioJack4") (at 254 71.12 0) (mirror y) (unit 1)
     (in_bom yes) (on_board yes) (dnp no) (fields_autoplaced)
-    (property "Reference" "J1" (at 256.54 63.5 0)
-      (effects (font (size 1.27 1.27)))
-    )
-    (property "Value" "Bridge" (at 256.54 66.04 0)
+    (property "Reference" "J1" (at 251.46 63.5 0)
+      (effects (font (size 1.27 1.27)))
+    )
+    (property "Value" "Bridge" (at 251.46 66.04 0)
       (effects (font (size 1.27 1.27)))
     )
@@
       (effects (font (size 1.27 1.27)) hide)
     )
-    (pin "R1")
-    (pin "R2")
+    (pin "RX")
+    (pin "TX")
     (pin "S")
     (pin "T")

Commit message: Add LEDs
Parts:
- added D1, D2, D3: LED, nantor:LED_0805, symbol Device:LED
- added R1, R2, R3: R, nantor:LED_0805, symbol Device:R
Connections:
- net GND: now also R1.1, R2.1, R3.1
- net L3: now reaches U1.1 (PB12)
- net L3: now also D3.2 (A)
- net TX: now reaches J1.TX, U1.14 (PB6)
- net RX: now reaches J1.RX, U1.15 (PB7)
- net BatActive: now reaches SW1.2 (B), SW2.2 (B), U1.21 (VBat)
- net L2: now reaches U1.6 (PA9)
- net L2: now also D2.2 (A)
- net L1: now reaches U1.7 (PA10)
- net L1: now also D1.2 (A)
- net BatPwr: now reaches J2.1 (Pin_1), SW1.1 (A), SW2.3 (C)
- new net: D1.1 (K), R1.2
- new net: D3.1 (K), R3.2
- new net: D2.1 (K), R2.2
- no-connect marks 14 -> 12
